File: src/dummyLoad/dummyLoad.brd (EAGLE design)
At the start: 49.5 x 49.5 mm, 34 parts, among them IC1 LM358D, Q1 MOSFET-NCHANNELPTH2, U1 LOAD POWER

Commit message: Minor updates to PCB and layout
Parts:
- moved R16 1.27 mm to (22.9, 26.7)
- moved C1 1.02 mm to (36.3, 2.79)
Routing:
- net N$4: track 4.33 -> 5.71 mm
- net N$7: track 6.36 -> 4.98 mm
- net VSENSE: track 31.5 -> 30.7 mm
Changed lines of the file:
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@@
 <?xml version="1.0" encoding="utf-8"?>
 <!DOCTYPE eagle SYSTEM "eagle.dtd">
-<eagle version="7.5.0">
+<eagle version="7.6.0">
 <drawing>
 <settings>
@@
 <layers>
 <layer number="1" name="Top" color="4" fill="1" visible="yes" active="yes"/>
-<layer number="16" name="Bottom" color="1" fill="1" visible="no" active="yes"/>
+<layer number="16" name="Bottom" color="1" fill="1" visible="yes" active="yes"/>
 <layer number="17" name="Pads" color="2" fill="1" visible="yes" active="yes"/>
 <layer number="18" name="Vias" color="2" fill="1" visible="yes" active="yes"/>
@@
 <attribute name="VALUE" x="38.354" y="-0.381" size="1.27" layer="27"/>
 </element>
-<element name="C1" library="rcl" package="C0805" value="0.1uF" x="36.322" y="3.81" smashed="yes" rot="R90">
-<attribute name="NAME" x="35.306" y="5.588" size="0.8128" layer="25" ratio="12" rot="R180"/>
-<attribute name="VALUE" x="38.862" y="2.54" size="1.27" layer="27" rot="R90"/>
+<element name="C1" library="rcl" package="C0805" value="0.1uF" x="36.322" y="2.794" smashed="yes" rot="R90">
+<attribute name="NAME" x="35.306" y="4.572" size="0.8128" layer="25" ratio="12" rot="R180"/>
+<attribute name="VALUE" x="38.862" y="1.524" size="1.27" layer="27" rot="R90"/>
 </element>
 <element name="C3" library="rcl" package="C0805" value="0.1uF" x="28.956" y="7.62" smashed="yes">
@@
 <attribute name="VALUE" x="17.272" y="4.318" size="0.8128" layer="27" ratio="12" rot="R270"/>
 </element>
-<element name="R16" library="resistor" package="M0805" value="100R" x="24.13" y="26.67" smashed="yes" rot="R90">
-<attribute name="NAME" x="25.4" y="29.464" size="0.8128" layer="25" ratio="12" rot="R180"/>
-<attribute name="VALUE" x="26.162" y="25.146" size="0.8128" layer="27" ratio="12" rot="R90"/>
+<element name="R16" library="resistor" package="M0805" value="100R" x="22.86" y="26.67" smashed="yes" rot="R90">
+<attribute name="NAME" x="24.13" y="29.464" size="0.8128" layer="25" ratio="12" rot="R180"/>
+<attribute name="VALUE" x="24.892" y="25.146" size="0.8128" layer="27" ratio="12" rot="R90"/>
 </element>
 <element name="C4" library="rcl" package="C0805" value="0.1uF" x="21.844" y="2.794" smashed="yes" rot="R90">
@@
 <via x="15.24" y="20.32" extent="1-16" drill="0.35"/>
 <via x="15.24" y="26.67" extent="1-16" drill="0.35"/>
-<via x="21.59" y="26.67" extent="1-16" drill="0.35"/>
+<via x="20.32" y="26.67" extent="1-16" drill="0.35"/>
 <via x="15.24" y="13.97" extent="1-16" drill="0.35"/>
 <via x="21.59" y="13.97" extent="1-16" drill="0.35"/>
@@
 <wire x1="23.2181" y1="11.938" x2="23.2181" y2="14.0741" width="0.3048" layer="1"/>
 <wire x1="23.2181" y1="14.0741" x2="23.495" y2="14.351" width="0.3048" layer="1"/>
-<wire x1="26.67" y1="1.016" x2="35.814" y2="1.016" width="0.3048" layer="1"/>
-<wire x1="35.814" y1="1.016" x2="36.322" y2="1.524" width="0.3048" layer="1"/>
-<wire x1="36.322" y1="1.524" x2="36.322" y2="2.86" width="0.3048" layer="1"/>
-<wire x1="36.322" y1="2.86" x2="39.558" y2="2.86" width="0.3048" layer="1"/>
-<wire x1="39.558" y1="2.86" x2="39.624" y2="2.794" width="0.3048" layer="1"/>
+<wire x1="26.67" y1="1.016" x2="34.036" y2="1.016" width="0.3048" layer="1"/>
+<wire x1="34.036" y1="1.016" x2="34.798" y2="1.778" width="0.3048" layer="1"/>
+<wire x1="34.798" y1="1.778" x2="36.256" y2="1.778" width="0.3048" layer="1"/>
+<wire x1="36.256" y1="1.778" x2="36.322" y2="1.844" width="0.3048" layer="1"/>
+<wire x1="39.624" y1="2.794" x2="38.608" y2="1.778" width="0.3048" layer="1"/>
+<wire x1="38.608" y1="1.778" x2="36.388" y2="1.778" width="0.3048" layer="1"/>
+<wire x1="36.388" y1="1.778" x2="36.322" y2="1.844" width="0.3048" layer="1"/>
 </signal>
 <signal name="N$2">
@@
 <contactref element="IC1" pad="7"/>
 <contactref element="R16" pad="1"/>
-<wire x1="24.13" y1="25.72" x2="24.13" y2="24.892" width="0.4064" layer="1"/>
-<wire x1="24.13" y1="24.892" x2="24.765" y2="24.257" width="0.4064" layer="1"/>
-<wire x1="24.765" y1="21.65" x2="24.765" y2="24.257" width="0.4064" layer="1"/>
+<wire x1="22.86" y1="25.72" x2="24.318" y2="25.72" width="0.4064" layer="1"/>
+<wire x1="24.318" y1="25.72" x2="24.765" y2="25.273" width="0.4064" layer="1"/>
+<wire x1="24.765" y1="21.65" x2="24.765" y2="25.273" width="0.4064" layer="1"/>
 </signal>
 <signal name="N$7">
 <contactref element="Q1" pad="1"/>
 <contactref element="R16" pad="2"/>
-<wire x1="24.13" y1="27.62" x2="22.672" y2="27.62" width="0.4064" layer="1"/>
-<wire x1="22.672" y1="27.62" x2="22.352" y2="27.94" width="0.4064" layer="1"/>
-<wire x1="22.352" y1="27.94" x2="22.352" y2="32.385" width="0.4064" layer="1"/>
+<wire x1="22.352" y1="32.385" x2="22.352" y2="29.718" width="0.4064" layer="1"/>
+<wire x1="22.352" y1="29.718" x2="22.86" y2="29.21" width="0.4064" layer="1"/>
+<wire x1="22.86" y1="29.21" x2="22.86" y2="27.62" width="0.4064" layer="1"/>
 </signal>
 </signals>
